File: SmartWatchRedux-E/SmartWatchRedux-E.sch (KiCad schematic (older format))
At the start: 6 parts, among them CN1 27C256Socket, U1 ROM, U2 DS1315, Y1 32.768 KHz

Commit message: Minor tweakes to board, add -E to name.
Parts:
- C1: footprint Capacitor_SMD:C_0805_2012Metric_Pad1.18x1.45mm_HandSolder -> Capacitor_SMD:C_1206_3216Metric
Changed lines of the file:
@@
 encoding utf-8
 Sheet 1 1
-Title "SmartWatch Redux"
+Title "SmartWatch Redux - E"
 Date ""
 Rev ""
@@
 F 0 "C1" H 3065 4396 50  0000 L CNN
 F 1 "0.1uF" H 3065 4305 50  0000 L CNN
-F 2 "Capacitor_SMD:C_0805_2012Metric_Pad1.18x1.45mm_HandSolder" H 2988 4200 50  0001 C CNN
+F 2 "Capacitor_SMD:C_1206_3216Metric" H 2988 4200 50  0001 C CNN
 F 3 "~" H 2950 4350 50  0001 C CNN
 	1    2950 4350
